File: sunbeam2.sch (EAGLE design)
At the start: 286 parts, among them IC10 LM1117IMPX-3.3, IC2 A4983, IC3 A4983, IC4 A4983, IC5 A4983, IC6 A4983, IC7 FT232RLSSOP, IC8 LM2675, IC9 LMV358MMX, Q1 BC857ALT1SMD, Q2 IRLHM630TR2PBF, Q3 IRLHM630TR2PBF, Q4 IRLHM630TR2PBF, T2 bc848, T3 bc858, T4 bc848, T5 bc858, T6 bc848, T7 bc858, U2 USD-SOCKETNEW

Commit message: -changed 3 2 channel pots to one 6 channel -moved play button -added fet driver for heater instead of bjts -changed some polygons [thanks triffin_hunter]
Parts:
- removed C80, C81: 0.1uF, rcl:C-EUC0603
- removed R84, R85: 15K, rcl:R-EU_R0603
- removed R86, R87, R92, R93: 10K, rcl:R-EU_R0603
- removed T2, T4, T6: bc848, transistor-neu-to92:BC848A-NPN-SOT23-BEC
- removed T3, T5, T7: bc858, transistor-neu-to92:BC858A-PNP-SOT23-BEC
- removed U$13, U$14, U$15: MCP4631, microchip:MCP4631
- added AD5206: AD5206, analog-devices:AD5206
- added C83, C84: 0.1uF, rcl:C-EUC0603
- added C85, C86: 4.7uF, rcl:C-EUC0603
- added FET_DRV1, FET_DRV2: TC4427, custom_esorensen:TC4427
- R76, R78, R80: value 1K -> 22R
- R77, R79, R81: value 1K -> 10K
- R83: value 15K -> 10K
- renumbered U$24 to E0_FET
Connections:
- removed net N$141: LPC1769.P4[29]/TX_MCLK/MAT2[1]/RXD3
- removed net N$161: R83.1, U$13.P0B, U$13.P1B
- removed net N$162: R84.1, U$14.P0B, U$14.P1B
- removed net N$163: R85.1, U$15.P0B, U$15.P1B
- removed net N$167: U$15.P0W
- removed net N$168: R86.1, U$14.A1
- removed net N$170: R87.1, U$15.A2
- new net N$148: AD5206.A1, AD5206.A2, AD5206.A3, AD5206.A4, AD5206.A6, R83.1
- new net POT_CS: AD5206.!CS, LPC1769.P4[29]/TX_MCLK/MAT2[1]/RXD3
- net +3V3: now also AD5206.VDD, C79.1; no longer C79.2, C80.2, C81.2, R84.2, R85.2, R86.2, R87.2, R92.2, R93.2, U$13.VDD, U$14.VDD, U$15.VDD
- net 5V: now also C83.1, C84.1, C85.1, C86.1, FET_DRV1RAILS.P$1, FET_DRV2RAILS.P$1; no longer T2.C, T4.C, T6.C
- net E0_H: now also FET_DRV1A.P$1; no longer T2.B, T3.B
- net E1_H: now also FET_DRV1B.P$1; no longer T4.B, T5.B
- net GND: now also AD5206.B1, AD5206.B2, AD5206.B3, AD5206.B4, AD5206.B6, AD5206.GND, AD5206.VSS, C79.2, C83.2, C84.2, C85.2, C86.2, FET_DRV1RAILS.P$2, FET_DRV2RAILS.P$2; no longer C79.1, C80.1, C81.1, T3.C, T5.C, T7.C, U$13.A1, U$13.A2, U$13.HVC/A0, U$13.P0A, U$13.P1A, U$13.VSS, U$14.A2, U$14.HVC/A0, U$14.P0A, U$14.P1A, U$14.VSS, U$15.A1, U$15.HVC/A0, U$15.P0A, U$15.P1A, U$15.VSS
- net HB_H: now also FET_DRV2A.P$1; no longer T6.B, T7.B
- net N$135: now also FET_DRV1B.P$2, R78.2; no longer R76.2, T2.E, T3.E
- net N$139: now also FET_DRV2A.P$2; no longer T6.E, T7.E
- net N$33: now also FET_DRV1A.P$2, R76.2; no longer R78.2, T4.E, T5.E
- net POT_SCL: no longer R92.1, U$13.SCL, U$14.SCL, U$15.SCL
- net POT_SDA: no longer R93.1, U$13.SDA, U$14.SDA, U$15.SDA
- net REF_E0: now also AD5206.W1; no longer U$14.P0W
- net REF_E1: now also AD5206.W3; no longer U$15.P1W
- net REF_X: now also AD5206.W6; no longer U$13.P1W
- net REF_Y: now also AD5206.W4; no longer U$13.P0W
- net REF_Z: now also AD5206.W2; no longer U$14.P1W
- net SD_MOSI: now also AD5206.SDI
- net SD_SCK: now also AD5206.CLK
Other:
- moved on the sheet: C79, E1-1, E1-2, E1_FET, HB-1, HB-2, HOTBET_FET, LED7, LED8, R76, R77, R78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

Commit message: -changed heaters fuse -some slight component changes
Parts:
- C15: value 1uF -> 0.1uF
- C23, C33, C40, C47, C54: value (none) -> 100uF
- D1: value 10BQ040PBF -> SS14; device diode:SCHOTTKY-DIODESMD -> diode:DIODE-DO214AC
- D2, D3: value (none) -> M4; device diode:DIODE-SMC -> diode:DIODE-DO214AC
- F4: value SMF_OMNIBLOK_154.062 -> 01530008Z; device _hhn_littlefuse_Nano2SMF_2:SMF_OMNIBLOK_154.062 -> Littelfuse_By_element14_Batch_1:01530008Z
- L2: device SparkFun:INDUCTOR0805 -> SparkFun:INDUCTOR0603
- PLAY, PROGRAM, RESET: device microbuilder:SWITCH_TACT_SMT -> SparkFun:TAC_SWITCHSMD
- R11, R28, R36, R44, R52: value R40 -> 10K
- R12, R13, R29, R30, R37, R38, R45, R46, R53, R54: value 0.2R -> 0.5R
- R3: value 50R -> 470R
- R90: value 5K -> 4K7
- T1: value (none) -> IRLML2246TRPBF
- renumbered U$5 to RJ1
Connections:
- removed net N$146: F3.1, V_MOT-1.KL
- new net N$117: F4.P$1, V_HEAT-2.KL
- net +3V3: now also C14.+; no longer C15.1
- net 5V: now also C15.1; no longer C14.+
- net GND: now also PLAY.3, PLAY.4, PROGRAM.3, PROGRAM.4, RESET.3, RESET.4, V_HEAT-1.KL, V_MOT-1.KL; no longer PLAY.S, PLAY.S1, PROGRAM.S, PROGRAM.S1, RESET.S, RESET.S1, V_HEAT-2.KL, V_MOT-2.KL
- net N$27: now also F3.1, V_MOT-2.KL; no longer F4.1, V_HEAT-1.KL
- net PLAY: now also PLAY.1, PLAY.2; no longer PLAY.P, PLAY.P1
- net PROGRAM: now also PROGRAM.1, PROGRAM.2; no longer PROGRAM.P, PROGRAM.P1
- net RESET: now also RESET.1, RESET.2; no longer RESET.P, RESET.P1
- net V_EXTR: now also F4.P$2; no longer F4.2
Other:
- moved on the sheet: C14, C15, V_HEAT-1, V_HEAT-2, V_MOT-1, V_MOT-2
